File: 4x3 keyboard/3x4 keyboard.kicad_pcb (KiCad board)
At the start: 2 copper layers, 60 x 55 mm, 33 parts, among them J1 Groove, SW1 SW_Push, SW10 SW_Push, SW11 SW_Push, SW12 SW_Push, SW2 SW_Push, SW3 SW_Push, SW4 SW_Push, SW5 SW_Push, SW6 SW_Push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

Commit message: Finishing touches and a readme
Parts:
- removed U2: MCP1700x-330xxTT, Package_TO_SOT_SMD:SOT-23
- added U3: ME6211C33M5, Package_TO_SOT_SMD:SOT-23-5, B.Cu at (125.5, 86.0)
- moved C1 3.94 mm to (127.5, 89.5)
- moved C3 2.98 mm to (123.5, 89.5), turned to 180 degrees
- moved R3 1.51 mm to (123.5, 93.0)
- moved TP1 1.51 mm to (120.5, 94.0)
Routing:
- net GND: track 3.06 -> 11.1 mm, vias 1 -> 2
- net VCC: track 11.4 -> 18.2 mm
- net /RST: track 8.17 -> 8.96 mm
